File: Eagle/sfg_clone.brd (EAGLE design)
At the start: 134 x 121 mm, 121 parts, among them IC1 27C512AP, IC2 74LS04D, IC3 EPM7160-T100, IC4 YM2151, IC5 YM3012, IC6 LM4556N, IC7 LM4556N, IC8 LM4558N, IC9 TLP552, Q1 4mHz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

Commit message: The sources for v1.0 board
Routing:
- net BUSDIR: vias 1 -> 0
Changed lines of the file:
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@@
 <wire x1="11.5" y1="45.5" x2="10.21" y2="45.5" width="0.3" layer="1"/>
 <wire x1="10.21" y1="45.5" x2="8.96" y2="46.75" width="0.3" layer="1"/>
-<via x="49" y="56.17" extent="1-16" drill="0.6"/>
 </signal>
 <signal name="MREQ">
